File: BSPD 1002/BSPD 1002.kicad_pcb (KiCad board)
At the start: 2 copper layers, 58 x 78 mm, 55 parts, among them J1 12V Supply, J2 Sensors, J3 Sensors, J4 Relay Output, K1 Relay_SPST-NO, Q1 BSS205N, Q2 BSS205N, U1 TLV1704, U2 TLV1704, U3 CD4093BM96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

Commit message: "Ready to buy"
Parts:
- added G***: LOGO, Custom_MSM:Decorative_Stinger, B.Cu at (107.8, 104.5)
- added REF**: jamesp-F.Cu, CustomFootprints:jamesp-F.Cu, F.Cu at (132.8, 104.8)
- moved R12 19.6 mm to (140.2, 79.0)
- moved R11 18.9 mm to (140.2, 76.0)
- moved TP4 6.75 mm to (140.2, 101.0)
- moved R21 5.00 mm to (107.0, 106.0)
Routing:
- net +5V: track 0.00 -> 244.0 mm
- net Net-(R13-Pad2): track 0.00 -> 92.5 mm, vias 0 -> 4
- net Net-(Q1-G): track 0.00 -> 85.5 mm, vias 0 -> 2
- net +12V: track 0.00 -> 78.3 mm
- net Net-(R8-Pad2): track 0.00 -> 62.2 mm, vias 0 -> 3
- net Net-(R7-Pad2): track 0.00 -> 56.6 mm, vias 0 -> 4
- net Net-(U1D--): track 0.00 -> 37.0 mm
- net 2.27V_REF: track 0.00 -> 36.1 mm, vias 0 -> 3
- net SENS_2: track 0.00 -> 35.6 mm, vias 0 -> 2
- net Net-(U2A--): track 0.00 -> 35.0 mm, vias 0 -> 2
- net 0.45V_REF: track 0.00 -> 32.3 mm, vias 0 -> 3
- net Net-(U1A--): track 0.00 -> 32.0 mm
- net Net-(U2B--): track 0.00 -> 28.0 mm, vias 0 -> 2
- net Net-(R21-Pad1): track 0.00 -> 25.4 mm
- net SENS_1: track 0.00 -> 23.7 mm
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- added copper zone on B.Cu, net GND
- added copper zone on F.Cu, net GND
Other:
- board text added: "12V"
- board text added: "D1"
- board text added: "D2"
- board text added: "D3"
- board text added: "GND"
- board text added: "Manchester Stinger Motorsports Brake System Plausibility Device Routed 11/02/2026"
- board text added: "S1"
- board text added: "S2"
- board text added: "SCS"
- board text added: "SDC IN"
- board text added: "SDC OUT"
- board text added: "SENS1"
- board text added: "SENS2"
