File: BSPD/BSPD.kicad_pcb (KiCad board)
At the start: 2 copper layers, 58 x 78 mm, 56 parts, among them IC1 CD4093BMT, IC2 CD4093BMT, J1 12V Supply, J2 Sensors, J3 Sensors, J4 Relay Output, K1 Relay_SPST-NO, Q1 BSS205N, Q2 BSS205N, U1 TLV1704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

Commit message: ready to go
Parts:
- added REF**: jamesp-F.Cu, CustomFootprints:jamesp-F.Cu, F.Cu at (101.8, 84.5)
Connections:
- J1 pad 1: +12V -> GND
- J1 pad 2: GND -> +12V
- J2 pad 1: SENS_1 -> GND
- J2 pad 2: GND -> SENS_1
- J3 pad 1: SENS_2 -> GND
- J3 pad 2: GND -> SENS_2
Routing:
- net Sens 2 Checked: track 66.7 -> 61.7 mm
- net GND: vias 11 -> 16
Other:
- board text added: "Manchester Stinger Motorsports Brake System Plausibility Device Routed 09/06/2026"
- board text removed: "Manchester Stinger Motorsports Brake System Plausibility Device Routed 11/02/2026"
