File: BSPD/BSPD.kicad_pcb (KiCad board)
At the start: 2 copper layers, 58 x 78 mm, 57 parts, among them IC1 CD4093BMT, IC2 CD4093BMT, J1 12V Supply, J2 Sensors, J3 Sensors, J4 Relay Output, K1 Relay_SPST-NO, Q1 BSS205N, Q2 BSS205N, U1 TLV1704, U2 TLV1704, U5 BD450, U6 SE555DR

Commit message: Changed 555 Timer's N-Mosfet to P-mosfet
Parts:
- removed the REF** at (101.8, 84.5)
- Q1: value BSS205N -> BSS215P
Connections:
- C4 pad 1: Net-(Q1-D) -> Net-(Q1-S)
- R19 pad 2: Net-(Q1-S) -> Net-(Q1-D)
- R20 pad 1: Net-(Q1-D) -> Net-(Q1-S)
- U6 pad 6: Net-(Q1-D) -> Net-(Q1-S)
- U6 pad 7: Net-(Q1-D) -> Net-(Q1-S)
Routing:
- net Net-(Q1-D): track 23.2 -> 8.19 mm, vias 0 -> 2
- net Net-(Q1-S): track 3.38 -> 15.6 mm, vias 0 -> 2
- net Net-(Q1-G): track 85.5 -> 84.6 mm
- net Net-(Q2-G): track 3.34 -> 4.15 mm
