File: BSPD/BSPD.kicad_sch (KiCad schematic)
At the start: 54 parts, among them IC1 CD4093BMT, IC2 CD4093BMT, J1 12V Supply, J2 Sensors, J3 Sensors, J4 Relay Output, K1 Relay_SPST-NO, Q1 BSS205N, Q2 BSS205N, U1 TLV1704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

Commit message: ready to go
Connections:
- net +12V: now also J1.2 (Pin_2); no longer J1.1 (Pin_1)
- net GND: now also J1.1 (Pin_1), J2.1 (Pin_1), J3.1 (Pin_1); no longer J1.2 (Pin_2), J2.2 (Pin_2), J3.2 (Pin_2)
- net SENS_1: now also J2.2 (Pin_2); no longer J2.1 (Pin_1)
- net SENS_2: now also J3.2 (Pin_2); no longer J3.1 (Pin_1)
Other:
- moved on the sheet: J1, J2, J3
