File: BSPD/BSPD.kicad_sch (KiCad schematic)
At the start: 54 parts, among them IC1 CD4093BMT, IC2 CD4093BMT, J1 12V Supply, J2 Sensors, J3 Sensors, J4 Relay Output, K1 Relay_SPST-NO, Q1 BSS205N, Q2 BSS205N, U1 TLV1704, U2 TLV1704, U5 BD450, U6 SE555DR

Commit message: Changed 555 Timer's N-Mosfet to P-mosfet
Parts:
- removed Q1: BSS205N, Custom_MSM:MOSFET_Single_SOT-23, symbol Custom_MSM:MOSFET_N-CH
- added Q1: BSS215P, Custom_MSM:MOSFET_Single_SOT-23, symbol Custom_MSM1:MOSFET_P-CH
Connections:
- net at R18.2, TP4.1, U1.14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: now also Q1.1 (G)
- net at R19.2: now also Q1.3 (D)
- net at C4.1, R20.1, U6.6 (THR)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: now also Q1.2 (S)
Other:
- moved on the sheet: R15, TP3, TP5
